File: LM-Seat/LED-Controller/PCB/LED-Main-V3.2/LED-Main-V3.2.kicad_pcb (KiCad board)
At the start: 2 copper layers, 190 x 100.6 mm, 141 parts, among them J1 5267-04P, J11 5267-04P, J15 Conn_01x03_Pin, J2 Conn_01x14_Pin, J3 Conn_01x02_Pin, J4 5267-04P, J7 5267-04P, J9 ECH381V-2P, K1 SIP-1B12, K3 DC12V-A, K5 DC12V-A, M1 Fan, Q1 AOD4185, Q10 AOD4185, Q11 AOD4185, Q12 AOD4185, Q13 AOD4185, Q16 AO3400A, Q17 MMBTA42L, Q18 MMBTA42L, Q19 AOD4185, Q2 AOD4185, Q20 AOD4185, Q3 MMBTA42L, Q5 MMBTA42L, Q6 AOD4185, Q7 AOD4185, Q8 MMBTA42L, Q9 MMBTA42L, SW2 SW_Push, SW3 RST, SW4 BOOT, SW5 SW_Push, SW7 YSS-1203, SW8 NW3-SK-02, U1 3.3V, U2 ESP32-S3-PCB, U4 485

Commit message: 2025-03-09-20:42 commit
Connections:
- R37 pad 2: Net-(U2-IO_7) -> Net-(U2-IO_17)
- U2 pad 10: unconnected-(U2-IO_17-Pad10) -> Net-(U2-IO_17)
- U2 pad 7: Net-(U2-IO_7) -> unconnected-(U2-IO_7-Pad7)
Routing:
- net Net-(U2-IO_7): track 30.5 -> 0.00 mm, vias 2 -> 0
- net Net-(U2-IO_17): track 0.00 -> 26.5 mm, vias 0 -> 1
