File: LM-Seat/LED-Controller/PCB/LED-Main-V3.2/LED-Main-V3.2.kicad_sch (KiCad schematic)
At the start: 139 parts, among them J1 5267-04P, J1 ECH381V-2P, J11 5267-04P, J11 Conn_01x02_Pin, J11 Conn_01x03_Pin, J19 Conn_01x14_Pin, J4 5267-04P, J7 5267-04P, K1 SIP-1B12, K4 DC12V-A, Q16 AO3400A, Q18 MMBTA42L, Q19 AOD4185, Q20 AOD4185, Q22 MMBTA42L, Q27 AOD4185, Q28 AOD4185, SW12 SW_Push, SW3 RST, SW4 BOOT, SW7 YSS-1203, SW8 NW3-SK-02, U1 3.3V, U2 485, U2 ESP32-S3-PCB

Commit message: 2025-03-09-20:42 commit
Connections:
- net at U2.10 (IO_17): now also R37.2
- net at U2.7 (IO_7): no longer R37.2
Changed lines of the file:
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@@
 	(wire
 		(pts
-			(xy 171.45 128.27) (xy 171.45 107.95)
+			(xy 171.45 128.27) (xy 171.45 115.57)
 		)
 		(stroke
@@
 	(wire
 		(pts
+			(xy 171.45 115.57) (xy 185.42 115.57)
+		)
+		(stroke
+			(width 0)
+			(type default)
+		)
+	)
+	(wire
+		(pts
 			(xy 42.672 168.275) (xy 42.672 203.708)
 		)
@@
 		)
 		(stroke
-			(width 0)
-			(type default)
-		)
-	)
-	(wire
-		(pts
-			(xy 171.45 107.95) (xy 185.42 107.95)
-		)
-		(stroke
